File: kicad/pong-retrosc.kicad_sch (KiCad schematic)
At the start: 24 parts, among them J1 RCA video (na placa), J4 chave A/B (painel), J5 pot P1 (painel), J6 pot P2 (painel), J7 START (painel), J8 RCA audio L (na placa), J9 RCA audio R (na placa), SW1 START, SW2 A/B, U1 RaspberryPi_Pico, U2 PAM8403 HW-012

Commit message: kicad: placa 55x88 refeita com feedback de revisao (DRC 0 erros)
- PAM8403: barra real de 11 posicoes (4+vazio+2+vazio+3), corpo na placa
  ao lado do USB e pot de volume saindo pela borda superior
- Pico com o USB colado na borda para facilitar o cabo no gabinete
- RCAs com o barril protraindo ~8,5 mm para fora da borda direita
- headers empilhados com nome e funcao de cada pino no silk; J5+J6 na
  mesma fileira com 1 vaga (aceita conector femea 1x7 unico)
- furos M3 regulares: base H2/H4/H3 em y84 (H2-H3 = 45 mm, H4 central)
  e H1 no eixo, 45 mm acima de H4
- logo RetroSC no silk da frente, entre as fileiras do Pico (0,22 mm/px)
- gerbers + pong-retrosc-gerbers.zip prontos para a fabrica

Co-Authored-By: Claude Opus 4.8 <noreply@anthropic.com>
Parts:
- R1, R2, R3, R4, R5, R6, R7: footprint Resistor_THT:R_Axial_DIN0207_L6.3mm_D2.5mm_P10.16mm_Horizontal -> Resistor_THT:R_Axial_DIN0207_L6.3mm_D2.5mm_P2.54mm_Vertical
Changed lines of the file:
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@@
 		(instances
 			(project "pong-retrosc"
-				(path "/54382c2c-30b3-43b0-8332-7c9095b4b1c1"
+				(path "/84d51f01-d374-488c-b3c5-dd73d073b153"
 					(reference "U1")
 					(unit 1)
@@
 			)
 		)
-		(property "Footprint" "Resistor_THT:R_Axial_DIN0207_L6.3mm_D2.5mm_P10.16mm_Horizontal"
+		(property "Footprint" "Resistor_THT:R_Axial_DIN0207_L6.3mm_D2.5mm_P2.54mm_Vertical"
 			(at 132.08 40.64 0)
 			(hide yes)
@@
 		(instances
 			(project "pong-retrosc"
-				(path "/54382c2c-30b3-43b0-8332-7c9095b4b1c1"
+				(path "/84d51f01-d374-488c-b3c5-dd73d073b153"
 					(reference "R1")
 					(unit 1)
@@
 			)
 		)
-		(property "Footprint" "Resistor_THT:R_Axial_DIN0207_L6.3mm_D2.5mm_P10.16mm_Horizontal"
+		(property "Footprint" "Resistor_THT:R_Axial_DIN0207_L6.3mm_D2.5mm_P2.54mm_Vertical"
 			(at 157.48 40.64 0)
 			(hide yes)
@@
 		(instances
 			(project "pong-retrosc"
-				(path "/54382c2c-30b3-43b0-8332-7c9095b4b1c1"
+				(path "/84d51f01-d374-488c-b3c5-dd73d073b153"
 					(reference "R2")
 					(unit 1)
@@
 		(instances
 			(project "pong-retrosc"
-				(path "/54382c2c-30b3-43b0-8332-7c9095b4b1c1"
+				(path "/84d51f01-d374-488c-b3c5-dd73d073b153"
 					(reference "J1")
 					(unit 1)
@@
 			)
 		)
-		(property "Footprint" "Resistor_THT:R_Axial_DIN0207_L6.3mm_D2.5mm_P10.16mm_Horizontal"
+		(property "Footprint" "Resistor_THT:R_Axial_DIN0207_L6.3mm_D2.5mm_P2.54mm_Vertical"
 			(at 132.08 91.44 0)
 			(hide yes)
@@
 		(instances
 			(project "pong-retrosc"
-				(path "/54382c2c-30b3-43b0-8332-7c9095b4b1c1"
+				(path "/84d51f01-d374-488c-b3c5-dd73d073b153"
 					(reference "R3")
 					(unit 1)
@@
 		(instances
 			(project "pong-retrosc"
-				(path "/54382c2c-30b3-43b0-8332-7c9095b4b1c1"
+				(path "/84d51f01-d374-488c-b3c5-dd73d073b153"
 					(reference "C1")
 					(unit 1)
@@
 		(instances
 			(project "pong-retrosc"
-				(path "/54382c2c-30b3-43b0-8332-7c9095b4b1c1"
+				(path "/84d51f01-d374-488c-b3c5-dd73d073b153"
 					(reference "C2")
 					(unit 1)
@@
 			)
 		)
-		(property "Footprint" "Resistor_THT:R_Axial_DIN0207_L6.3mm_D2.5mm_P10.16mm_Horizontal"
+		(property "Footprint" "Resistor_THT:R_Axial_DIN0207_L6.3mm_D2.5mm_P2.54mm_Vertical"
 			(at 203.2 91.44 0)
 			(hide yes)
@@
 		(instances
 			(project "pong-retrosc"
-				(path "/54382c2c-30b3-43b0-8332-7c9095b4b1c1"
+				(path "/84d51f01-d374-488c-b3c5-dd73d073b153"
 					(reference "R4")
 					(unit 1)
@@
 			)
 		)
-		(property "Footprint" "Resistor_THT:R_Axial_DIN0207_L6.3mm_D2.5mm_P10.16mm_Horizontal"
+		(property "Footprint" "Resistor_THT:R_Axial_DIN0207_L6.3mm_D2.5mm_P2.54mm_Vertical"
 			(at 223.52 104.14 0)
 			(hide yes)
@@
 		(instances
 			(project "pong-retrosc"
-				(path "/54382c2c-30b3-43b0-8332-7c9095b4b1c1"
+				(path "/84d51f01-d374-488c-b3c5-dd73d073b153"
 					(reference "R5")
 					(unit 1)
@@
 			)
 		)
-		(property "Footprint" "Resistor_THT:R_Axial_DIN0207_L6.3mm_D2.5mm_P10.16mm_Horizontal"
+		(property "Footprint" "Resistor_THT:R_Axial_DIN0207_L6.3mm_D2.5mm_P2.54mm_Vertical"
 			(at 259.08 91.44 0)
 			(hide yes)
@@
 		(instances
 			(project "pong-retrosc"
-				(path "/54382c2c-30b3-43b0-8332-7c9095b4b1c1"
+				(path "/84d51f01-d374-488c-b3c5-dd73d073b153"
 					(reference "R6")
 					(unit 1)
@@
 			)
 		)
-		(property "Footprint" "Resistor_THT:R_Axial_DIN0207_L6.3mm_D2.5mm_P10.16mm_Horizontal"
+		(property "Footprint" "Resistor_THT:R_Axial_DIN0207_L6.3mm_D2.5mm_P2.54mm_Vertical"
 			(at 259.08 106.68 0)
 			(hide yes)
@@
 		(instances
 			(project "pong-retrosc"
-				(path "/54382c2c-30b3-43b0-8332-7c9095b4b1c1"
+				(path "/84d51f01-d374-488c-b3c5-dd73d073b153"
 					(reference "R7")
 					(unit 1)
@@
 		(instances
 			(project "pong-retrosc"
-				(path "/54382c2c-30b3-43b0-8332-7c9095b4b1c1"
+				(path "/84d51f01-d374-488c-b3c5-dd73d073b153"
 					(reference "U2")
 					(unit 1)
@@
 		(instances
 			(project "pong-retrosc"
-				(path "/54382c2c-30b3-43b0-8332-7c9095b4b1c1"
+				(path "/84d51f01-d374-488c-b3c5-dd73d073b153"
 					(reference "RV1")
 					(unit 1)
@@
 		(instances
 			(project "pong-retrosc"
-				(path "/54382c2c-30b3-43b0-8332-7c9095b4b1c1"
+				(path "/84d51f01-d374-488c-b3c5-dd73d073b153"
 					(reference "C3")
 					(unit 1)
@@
 		(instances
 			(project "pong-retrosc"
-				(path "/54382c2c-30b3-43b0-8332-7c9095b4b1c1"
+				(path "/84d51f01-d374-488c-b3c5-dd73d073b153"
 					(reference "J5")
 					(unit 1)
@@
 		(instances
 			(project "pong-retrosc"
-				(path "/54382c2c-30b3-43b0-8332-7c9095b4b1c1"
+				(path "/84d51f01-d374-488c-b3c5-dd73d073b153"
 					(reference "RV2")
 					(unit 1)
@@
 		(instances
 			(project "pong-retrosc"
-				(path "/54382c2c-30b3-43b0-8332-7c9095b4b1c1"
+				(path "/84d51f01-d374-488c-b3c5-dd73d073b153"
 					(reference "C4")
 					(unit 1)
@@
 		(instances
 			(project "pong-retrosc"
-				(path "/54382c2c-30b3-43b0-8332-7c9095b4b1c1"
+				(path "/84d51f01-d374-488c-b3c5-dd73d073b153"
 					(reference "J6")
 					(unit 1)
@@
 		(instances
 			(project "pong-retrosc"
-				(path "/54382c2c-30b3-43b0-8332-7c9095b4b1c1"
+				(path "/84d51f01-d374-488c-b3c5-dd73d073b153"
 					(reference "SW1")
 					(unit 1)
@@
 		(instances
 			(project "pong-retrosc"
-				(path "/54382c2c-30b3-43b0-8332-7c9095b4b1c1"
+				(path "/84d51f01-d374-488c-b3c5-dd73d073b153"
 					(reference "J7")
 					(unit 1)
@@
 		(instances
 			(project "pong-retrosc"
-				(path "/54382c2c-30b3-43b0-8332-7c9095b4b1c1"
+				(path "/84d51f01-d374-488c-b3c5-dd73d073b153"
 					(reference "J4")
 					(unit 1)
@@
 		(instances
 			(project "pong-retrosc"
-				(path "/54382c2c-30b3-43b0-8332-7c9095b4b1c1"
+				(path "/84d51f01-d374-488c-b3c5-dd73d073b153"
 					(reference "SW2")
 					(unit 1)
@@
 		(instances
 			(project "pong-retrosc"
-				(path "/54382c2c-30b3-43b0-8332-7c9095b4b1c1"
+				(path "/84d51f01-d374-488c-b3c5-dd73d073b153"
 					(reference "SW2")
 					(unit 2)
@@
 		(instances
 			(project "pong-retrosc"
-				(path "/54382c2c-30b3-43b0-8332-7c9095b4b1c1"
+				(path "/84d51f01-d374-488c-b3c5-dd73d073b153"
 					(reference "J8")
 					(unit 1)
@@
 		(instances
 			(project "pong-retrosc"
-				(path "/54382c2c-30b3-43b0-8332-7c9095b4b1c1"
+				(path "/84d51f01-d374-488c-b3c5-dd73d073b153"
 					(reference "J9")
 					(unit 1)
